File: Squid.kicad_sch (KiCad schematic)
At the start: 3 parts

Commit message: Обновил схемотехнику у платы. Убрал лишнее компоненты и лишнии линии
Parts:
- added R83, R84: 10, Resistor_SMD:R_0805_2012Metric, symbol Device:R
Connections:
- net USART2_RX: now also R83.1
- net USART2_TX: now also R84.1
- net RP_BOOT0: no longer names the net of RP1.16 (GPIO23)
- net RP_RST: no longer names the net of RP1.15 (GPIO22)
- net RP_RST: no longer SWD1.5 (Pin_5)
- net SPI1_CLK renamed SPI2_CLK
- net SPI1_MISO renamed SPI2_MOSI
- net SPI1_MOSI renamed SPI2_MISO
- net SPI1_NSS renamed SPI2_NSS
- new net NRST: SWD1.5 (Pin_5)
- new net sheet_set/MAIN_USART_RX: R83.2
- new net sheet_set/MAIN_USART_TX: R84.2
- no-connect marks 20 -> 49
Other:
- added sheet EndStopper1 (schematics/EndStopper.kicad_sch)
- added sheet EndStopper2 (schematics/EndStopper.kicad_sch)
- added sheet EndStopper3 (schematics/EndStopper.kicad_sch)
- added sheet EndStopper4 (schematics/EndStopper.kicad_sch)
- added sheet EndStopper5 (schematics/EndStopper.kicad_sch)
- added sheet EndStopper6 (schematics/EndStopper.kicad_sch)
- sheet STM32F407VG ports: added PH0, PH1; removed BOOT0, PA8
- sheet sheet_set ports: added M10_EN, M10_KEY, M10_SELECT, M10_STATUS; removed M0_BOOT0, M0_EN, M0_ENDSTOP_B, M0_KEY, M0_NRST, M0_SELECT, M0_STATUS, M1_BOOT0, M1_ENDSTOP_B, M1_NRST, M2_BOOT0, M2_ENDSTOP_B, M2_NRST, M3_BOOT0, M3_ENDSTOP_B, M3_NRST, M4_BOOT0, M4_ENDSTOP_B, M4_NRST, M5_BOOT0, M5_ENDSTOP_B, M5_NRST, M6_BOOT0, M6_ENDSTOP_B, M6_NRST, M7_BOOT0, M7_ENDSTOP_B, M7_NRST, M8_BOOT0, M8_ENDSTOP_B, M8_NRST, M9_BOOT0, M9_ENDSTOP_B, M9_NRST
- company: (none) -> МГТУ им. Н.Э.Баумана

Commit message: Обновлена нумерация элементов
Parts:
- renumbered R84 to R1, R83 to R2
Changed lines of the file:
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@@
 	(title_block
 		(title "Плата управления\\nшаговыми двигателями")
-		(date "2025-08-24")
+		(date "2025-08-25")
 		(company "МГТУ им. Н.Э.Баумана")
 		(comment 1 "БИГЕ.351101.001 Э3")
@@
 		(dnp no)
 		(fields_autoplaced yes)
-		(property "Reference" "#PWR04"
+		(property "Reference" "#PWR03"
 			(at 63.5 204.47 0)
 			(effects
@@
 			(project "MasterBoard"
 				(path "/97e8f341-b455-4614-ab7f-cc310164e7aa"
-					(reference "#PWR04")
+					(reference "#PWR03")
 					(unit 1)
 				)
@@
 		(on_board yes)
 		(dnp no)
-		(property "Reference" "R83"
+		(property "Reference" "R2"
 			(at 265.5584 20.2006 90)
 			(effects
@@
 			(project "Squid"
 				(path "/97e8f341-b455-4614-ab7f-cc310164e7aa"
-					(reference "R83")
+					(reference "R2")
 					(unit 1)
 				)
@@
 		(dnp no)
 		(fields_autoplaced yes)
-		(property "Reference" "#PWR03"
+		(property "Reference" "#PWR02"
 			(at 62.23 129.54 0)
 			(effects
@@
 			(project "MasterBoard"
 				(path "/97e8f341-b455-4614-ab7f-cc310164e7aa"
-					(reference "#PWR03")
+					(reference "#PWR02")
 					(unit 1)
 				)
@@
 		(dnp no)
 		(fields_autoplaced yes)
-		(property "Reference" "#PWR05"
+		(property "Reference" "#PWR04"
 			(at 64.77 129.54 0)
 			(effects
@@
 			(project "MasterBoard"
 				(path "/97e8f341-b455-4614-ab7f-cc310164e7aa"
-					(reference "#PWR05")
+					(reference "#PWR04")
 					(unit 1)
 				)
@@
 		(dnp no)
 		(fields_autoplaced yes)
-		(property "Reference" "#PWR02"
+		(property "Reference" "#PWR05"
 			(at 69.088 58.674 0)
 			(effects
@@
 			(project "MasterBoard"
 				(path "/97e8f341-b455-4614-ab7f-cc310164e7aa"
-					(reference "#PWR02")
+					(reference "#PWR05")
 					(unit 1)
 				)
@@
 		(on_board yes)
 		(dnp no)
-		(property "Reference" "R84"
+		(property "Reference" "R1"
 			(at 265.4834 30.2459 90)
 			(effects
@@
 			(project "Squid"
 				(path "/97e8f341-b455-4614-ab7f-cc310164e7aa"
-					(reference "R84")
+					(reference "R1")
 					(unit 1)
 				)
