File: schematics/STM32F407VG.kicad_sch (KiCad schematic)
At the start: 19 parts, among them SW1 SW_DPST_x2, U2 STM32F407VGTx, X1 8MHz

Commit message: Обновил схемотехнику у платы. Убрал лишнее компоненты и лишнии линии
Parts:
- removed C13, C14: 20p, Capacitor_SMD:C_0805_2012Metric, symbol Device:C
- removed C19: 4.7u, Capacitor_SMD:C_0805_2012Metric, symbol Device:C
- removed X1: 8MHz, Crystal:Crystal_HC49-U_Vertical, symbol Device:Crystal
- added LD36: CLK, LED_SMD:LED_0805_2012Metric, symbol Device:LED
- added R82: 10k, Resistor_SMD:R_0805_2012Metric, symbol Device:R
Connections:
- net +3.3V: now also R82.1
- net BOOT0: no longer names the net of R4.1, U2.94 (BOOT0)
- net OSC_IN renamed PH0
- net OSC_OUT renamed PH1
- net PA8: no longer names the net of U2.67 (PA8)
- net PA8: now also LD36.1 (K)
- new net: LD36.2 (A), R82.2
Other:
- company: (none) -> МГТУ им. Н.Э.Баумана

Commit message: Обновлена нумерация элементов
Parts:
- renumbered C15 to C13, C16 to C14, C17 to C15, C18 to C16, LD36 to LD3, R3 to R5, R4 to R6, R82 to R7
Changed lines of the file:
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@@
 	(title_block
 		(title "Плата управления\\nшаговыми двигателями")
-		(date "2025-02-17")
+		(date "2025-08-25")
 		(company "МГТУ им. Н.Э.Баумана")
 		(comment 1 "БИГЕ.351101.001 Э3")
@@
 		(on_board yes)
 		(dnp no)
-		(property "Reference" "R4"
+		(property "Reference" "R6"
 			(at 57.15 42.926 0)
 			(effects
@@
 			(project "stm32f4_ILI_RS_SD"
 				(path "/97e8f341-b455-4614-ab7f-cc310164e7aa/8db3f3ed-0435-4018-8cfb-2b18cdc95e24"
-					(reference "R4")
+					(reference "R6")
 					(unit 1)
 				)
@@
 		(on_board yes)
 		(dnp no)
-		(property "Reference" "C15"
+		(property "Reference" "C13"
 			(at 218.44 133.985 0)
 			(effects
@@
 			(project "MasterBoard"
 				(path "/97e8f341-b455-4614-ab7f-cc310164e7aa/8db3f3ed-0435-4018-8cfb-2b18cdc95e24"
-					(reference "C15")
+					(reference "C13")
 					(unit 1)
 				)
@@
 		(on_board yes)
 		(dnp no)
-		(property "Reference" "R82"
+		(property "Reference" "R7"
 			(at 154.1282 46.99 90)
 			(effects
@@
 			(project "Squid"
 				(path "/97e8f341-b455-4614-ab7f-cc310164e7aa/8db3f3ed-0435-4018-8cfb-2b18cdc95e24"
-					(reference "R82")
+					(reference "R7")
 					(unit 1)
 				)
@@
 		(dnp no)
 		(fields_autoplaced yes)
-		(property "Reference" "C18"
+		(property "Reference" "C16"
 			(at 246.38 141.605 0)
 			(effects
@@
 			(project "stm32f4_ILI_RS_SD"
 				(path "/97e8f341-b455-4614-ab7f-cc310164e7aa/8db3f3ed-0435-4018-8cfb-2b18cdc95e24"
-					(reference "C18")
+					(reference "C16")
 					(unit 1)
 				)
@@
 		(dnp no)
 		(fields_autoplaced yes)
-		(property "Reference" "R3"
+		(property "Reference" "R5"
 			(at 44.45 24.1299 0)
 			(effects
@@
 			(project "MasterBoard"
 				(path "/97e8f341-b455-4614-ab7f-cc310164e7aa/8db3f3ed-0435-4018-8cfb-2b18cdc95e24"
-					(reference "R3")
+					(reference "R5")
 					(unit 1)
 				)
@@
 		(on_board yes)
 		(dnp no)
-		(property "Reference" "LD36"
+		(property "Reference" "LD3"
 			(at 142.2362 46.851 0)
 			(effects
@@
 			(project "Squid"
 				(path "/97e8f341-b455-4614-ab7f-cc310164e7aa/8db3f3ed-0435-4018-8cfb-2b18cdc95e24"
-					(reference "LD36")
+					(reference "LD3")
 					(unit 1)
 				)
@@
 		(dnp no)
 		(fields_autoplaced yes)
-		(property "Reference" "C16"
+		(property "Reference" "C14"
 			(at 227.33 141.605 0)
 			(effects
@@
 			(project "MasterBoard"
 				(path "/97e8f341-b455-4614-ab7f-cc310164e7aa/8db3f3ed-0435-4018-8cfb-2b18cdc95e24"
-					(reference "C16")
+					(reference "C14")
 					(unit 1)
 				)
@@
 		(dnp no)
 		(fields_autoplaced yes)
-		(property "Reference" "#PWR029"
+		(property "Reference" "#PWR028"
 			(at 242.5412 132.08 0)
 			(effects
@@
 			(project "MasterBoard"
 				(path "/97e8f341-b455-4614-ab7f-cc310164e7aa/8db3f3ed-0435-4018-8cfb-2b18cdc95e24"
-					(reference "#PWR029")
+					(reference "#PWR028")
 					(unit 1)
 				)
@@
 		(on_board yes)
 		(dnp no)
-		(property "Reference" "C17"
+		(property "Reference" "C15"
 			(at 237.49 133.985 0)
 			(effects
@@
 			(project "stm32f4_ILI_RS_SD"
 				(path "/97e8f341-b455-4614-ab7f-cc310164e7aa/8db3f3ed-0435-4018-8cfb-2b18cdc95e24"
-					(reference "C17")
+					(reference "C15")
 					(unit 1)
 				)
@@
 		(dnp no)
 		(fields_autoplaced yes)
-		(property "Reference" "#PWR0214"
+		(property "Reference" "#PWR026"
 			(at 162.1552 54.4714 0)
 			(effects
@@
 			(project "Squid"
 				(path "/97e8f341-b455-4614-ab7f-cc310164e7aa/8db3f3ed-0435-4018-8cfb-2b18cdc95e24"
-					(reference "#PWR0214")
+					(reference "#PWR026")
 					(unit 1)
 				)
