File: schematics/power.kicad_sch (KiCad schematic)
At the start: 10 parts, among them U1 RT9193-33GB

Commit message: Обновил схемотехнику у платы. Убрал лишнее компоненты и лишнии линии
Other:
- company: (none) -> МГТУ им. Н.Э.Баумана
Changed lines of the file:
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@@
 	(title_block
 		(title "Плата управления\\nшаговыми двигателями")
-		(comment 1 "Питание")
+		(company "МГТУ им. Н.Э.Баумана")
+		(comment 1 "БИГЕ.351101.001 Э3")
 		(comment 2 "Филимонов С.В.")
+		(comment 3 "Семеренко Д.А.")
 	)
 	(text "+5V to +3.3V"

Commit message: Обновлена нумерация элементов
Parts:
- renumbered R1 to R3, R2 to R4
Changed lines of the file:
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@@
 	(title_block
 		(title "Плата управления\\nшаговыми двигателями")
+		(date "2025-08-25")
 		(company "МГТУ им. Н.Э.Баумана")
 		(comment 1 "БИГЕ.351101.001 Э3")
@@
 		(on_board yes)
 		(dnp no)
-		(property "Reference" "R2"
+		(property "Reference" "R4"
 			(at 143.51 121.92 90)
 			(effects
@@
 			(project "MasterBoard"
 				(path "/97e8f341-b455-4614-ab7f-cc310164e7aa/7330fb6d-3de7-4c19-a7a3-dd8fb4865426"
-					(reference "R2")
+					(reference "R4")
 					(unit 1)
 				)
@@
 		(on_board yes)
 		(dnp no)
-		(property "Reference" "R1"
+		(property "Reference" "R3"
 			(at 143.51 113.03 90)
 			(effects
@@
 			(project "MasterBoard"
 				(path "/97e8f341-b455-4614-ab7f-cc310164e7aa/7330fb6d-3de7-4c19-a7a3-dd8fb4865426"
-					(reference "R1")
-					(unit 1)
-				)
+					(reference "R3")
+					(unit 1)
+				)
