File: schematics/EndStopper.kicad_sch (KiCad schematic)
At the start: 4 parts

Commit message: Переименновал разъемы
Parts:
- ESC1: renamed from ESA12; value ESA -> ESC
- renumbered C66 to C57, R87 to R184, R88 to R185
